File: automedon/automedon.kicad_sch (KiCad schematic)
At the start: 8 parts, among them J1 701W-X2/03, J13 ZP-PNA-06-101, J16 Antenna, J2 MS3102E14S-2P, J3 MS3102E14S-2S, J4 MS3102E14S-2S, J5 MS3102E14S-2P, J6 MS3102E14S-2S

Commit message: Schematic ~70% done
Parts:
- removed J3, J4, J6: MS3102E14S-2S, symbol Connector:Conn_01x04_Socket
- removed J5: MS3102E14S-2P, symbol Connector:Conn_01x04_Pin
- added J3, J4, J45: PWM-02RMFS-TS7001, symbol Connector:Conn_01x02_Socket
- added MES1: Voltmeter Display, symbol Device:Voltmeter_DC
- added SW1: ELW115A12, symbol Switch:SW_SPST
- added SW3: SW_SPST, symbol Switch:SW_SPST
- J2: value MS3102E14S-2P -> MS3100E24-22P
Connections:
- net Valve Igniter Control/KEYSW+: now also SW3.1 (A)
- net Valve Igniter Control/KEYSW-: now also SW3.2 (B)
- net power/L: now also SW1.2 (B); no longer J1.1 (Pin_1)
- net tank_heating/BATT_24+: now also J45.1 (Pin_1)
- net tank_heating/BATT_24-: now also J45.2 (Pin_2)
- net tank_heating/TH1+: now also J3.1 (Pin_1)
- net tank_heating/TH1-: now also J3.2 (Pin_2)
- net tank_heating/TH2+: now also J4.1 (Pin_1)
- net tank_heating/TH2-: now also J4.2 (Pin_2)
- net power/BATT1+ renamed 1-BATT-01
- net power/BATT1- renamed 1-BATT-03
- net power/BATT2+ renamed 1-BATT-02
- net power/BATT2- renamed 1-BATT-04
- net power/N renamed 1-N-01
- new net 1-120-01: J1.1 (Pin_1), SW1.1 (A)
- new net power/VM_+: MES1.2 (+)
- new net power/VM_-: MES1.1 (-)
Other:
- sheet Valve Igniter Control ports: added RLCS_ETH; removed UART_RX, UART_TX
- sheet power ports: added VM_+, VM_-; removed none
- sheet tank_heating ports: added none; removed TH3+, TH3-
- note added: "*Rated to 15A but IP67"
- note added: "Apply liberal caulk"
- note added: "Take existing keyswitch so it matches Clientside Apply liberal caulk"
- note added: "mates PWM-02BFMB-TL7001"
- note added: "should mate w/ MS3106A24-22S w/ M85049/52-1-24W for strain relief [DOUBLE CHECK THESE]"
- moved on the sheet: J1, J2
