File: automedon/daq.kicad_sch (KiCad schematic)
At the start: 16 parts, among them J17 09-4224-00-04, J18 09-4224-00-04, J19 09-4224-00-04, J20 09-4224-00-04, J21 09-4224-00-04, J22 09-4224-00-04, J23 09-4224-00-04, J24 09-4224-00-04, J25 09-4224-00-04, J26 09-4224-00-04, J27 09-4224-00-04, J28 09-4224-00-04

Commit message: Schematic ~70% done
Other:
- note added: "RasPi"
Changed lines of the file:
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@@
+		)
+	)
+	(rectangle
+		(start 233.045 221.615)
+		(end 280.035 267.97)
+		(stroke
+			(width 0)
+			(type default)
+		)
+		(fill
+			(type none)
+		)
+	)
+	(text "RasPi"
+		(exclude_from_sim no)
+		(at 252.476 234.696 0)
+		(effects
+			(font
+				(size 1.27 1.27)
+			)
 		)
 	)
@@
 	)
 	(symbol
-		(lib_name "automedon:patch_panel")
 		(lib_id "automedon:patch_panel")
 		(at 306.07 161.29 0)
@@
 	)
 	(symbol
-		(lib_name "automedon:patch_panel")
 		(lib_id "automedon:patch_panel")
 		(at 306.07 49.53 0)
@@
 	)
 	(symbol
-		(lib_name "automedon:patch_panel")
 		(lib_id "automedon:patch_panel")
 		(at 306.07 87.63 0)
@@
 	)
 	(symbol
-		(lib_name "automedon:patch_panel")
 		(lib_id "automedon:patch_panel")
 		(at 306.07 124.46 0)
