File: automedon/ethernet.kicad_sch (KiCad schematic)
At the start: 2 parts

Commit message: Schematic ~70% done
Connections:
- new net: U10. (GND), U11. (VIN-)
- new net ETH_PI: U11. (VIN-)
- no-connect marks 1 -> 0
Other:
- note added: "2W @ 12V"
- note added: "Ubiquiti LiteBeam takes max 0.3A @ 24V"
Changed lines of the file:
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@@
 	(generator_version "8.0")
 	(paper "A4")
-	(no_connect
-		(at 114.3 93.98)
-	)
 	(wire
 		(pts
@@
 	(wire
 		(pts
+			(xy 115.57 93.98) (xy 114.3 93.98)
+		)
+		(stroke
+			(width 0)
+			(type default)
+		)
+	)
+	(wire
+		(pts
 			(xy 115.57 86.36) (xy 114.3 86.36)
 		)
@@
 		)
 	)
+	(text "2W @ 12V"
+		(exclude_from_sim no)
+		(at 103.632 99.06 0)
+		(effects
+			(font
+				(size 1.27 1.27)
+			)
+		)
+	)
+	(text "Ubiquiti LiteBeam takes max 0.3A @ 24V"
+		(exclude_from_sim no)
+		(at 164.338 94.996 0)
+		(effects
+			(font
+				(size 1.27 1.27)
+			)
+		)
+	)
 	(text "SE-SW5U-WT"
 		(exclude_from_sim no)
@@
 		(effects
 			(font
+				(size 1.27 1.27)
+			)
+			(justify left)
+		)
+	)
+	(hierarchical_label "ETH_PI"
+		(shape input)
+		(at 115.57 93.98 0)
+		(effects
+			(font
