File: automedon/power.kicad_sch (KiCad schematic)
At the start: 5 parts, among them SW1 AC_ON

Commit message: Schematic ~70% done
Parts:
- removed SW1: AC_ON, symbol Switch:SW_SPST
- added J29, J30, J31, J32, J33, J34, J35, J36, J37, J38, J39, J40, J41, J42, J43, J44: 3211771, symbol automedon:CONN_TERM_3
- CB1: value CircuitBreaker_2P -> GMCBU-1B-16
- CB2: value CircuitBreaker_1P -> Mersen 40120G; symbol Device:CircuitBreaker_1P -> Device:Fuse
Connections:
- net +12V: now also J30.1 (Pin_3); no longer PS2. (GND)
- net +24V: now also J38.1 (Pin_3)
- net +5V: now also J40.1 (Pin_3)
- net GND: now also J34.1 (Pin_3); no longer PS2. (GND)
- net L: now also CB1.2
- net 2-12-02: now reaches PS1.6 (+Vout)
- net 2-12-02: now also J29.1 (Pin_3); no longer CB2.1
- net 2-120-02: now reaches CB1.1, PS1.1 (AC/L)
- net 2-120-03: now reaches CB1.3, PS1.2 (EARTH)
- new net: J34.1 (Pin_3), J35.1 (Pin_3), J36.1 (Pin_3), J37.1 (Pin_3), J42.1 (Pin_3), J44.1 (Pin_3)
- new net: J30.1 (Pin_3), J31.1 (Pin_3), J32.1 (Pin_3), J33.1 (Pin_3), J43.1 (Pin_3)
- new net: J38.1 (Pin_3), J39.1 (Pin_3)
- new net: J40.1 (Pin_3), J41.1 (Pin_3)
- new net 2-12-01: J29.1 (Pin_3), PS1.6 (+Vout)
- new net 2-12-03: CB2.1, J29.1 (Pin_3)
- new net 2-12-05: J30.1 (Pin_3), PS2. (GND)
- new net 2-GND-02: J35.1 (Pin_3), PS1.3 (MB_NO)
- new net 2-GND-03: J34.1 (Pin_3), PS2. (GND)
- new net 2-GND-04: J34.1 (Pin_3), PS2. (GND)
- new net VM_+: J30.1 (Pin_3)
- new net VM_-: J35.1 (Pin_3)
- no-connect marks 6 -> 42
Other:
- note added: "16A MCB Form B"
- note added: "24/5V distribution"
- note added: "24V@3A 5V@3A"
- note added: "30 A Class G e.g. Littelfuse SLC030"
- note added: "Phoenix Contact CLIPLINE PT P/N 3211771 Jumper P/N 3030213"
- note removed: "20A?"
- moved on the sheet: CB1, PS1, PS2
