File: automedon/tank_heating.kicad_sch (KiCad schematic)
At the start: 3 parts

Commit message: Schematic ~70% done
Connections:
- net at U3. (SDA/CANL): no longer U1. (SDA/CANL)
- new net: U1. (SDA/CANL), U3. (SDA/CANL) (x5)
- new net: U1.1 (P1), U3.1 (P1) (x2)
- new net: U1.1 (P1), U2. (VOUT) (x2)
- now unconnected: U3. (SDA/CANL), U3. (SDA/CANL), U3. (SDA/CANL), U3. (SDA/CANL)
Other:
- note added: "RPP"
Changed lines of the file:
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@@
 	(wire
 		(pts
-			(xy 66.04 82.55) (xy 77.47 82.55)
+			(xy 52.07 82.55) (xy 77.47 82.55)
 		)
 		(stroke
@@
 	(wire
 		(pts
-			(xy 66.04 78.74) (xy 77.47 78.74)
+			(xy 52.07 78.74) (xy 77.47 78.74)
 		)
 		(stroke
@@
 		)
 	)
+	(text "RPP"
+		(exclude_from_sim no)
+		(at 87.63 75.184 0)
+		(effects
+			(font
+				(size 1.27 1.27)
+			)
+		)
+	)
 	(text "THR2"
 		(exclude_from_sim no)
@@
 	(hierarchical_label "BATT_24-"
 		(shape input)
-		(at 66.04 82.55 180)
+		(at 52.07 82.55 180)
 		(effects
 			(font
@@
 	(hierarchical_label "BATT_24+"
 		(shape input)
-		(at 66.04 78.74 180)
+		(at 52.07 78.74 180)
 		(effects
 			(font
@@
 	)
 	(symbol
-		(lib_name "automedon:RLCS_RELAY")
 		(lib_id "automedon:RLCS_RELAY")
 		(at 171.45 55.88 0)
