File: automedon/valve_relays.kicad_sch (KiCad schematic)
At the start: 16 parts, among them J10 MS3102E14S-6S, J11 MS3102E14S-6S, J12 MS3102E14S-6S, J14 Conn_01x02_Pin, J15 Conn_01x02_Pin, J7 MS3102E14S-6S, J8 MS3102E14S-6S, J9 MS3102E14S-6S, SW2 SW_DPST_x2

Commit message: Schematic ~70% done
Parts:
- added U17: ~, symbol automedon:ETH_UART
Connections:
- net GND: now also U17. (TX)
- net UART_RX: now also U17. (TX)
- net UART_TX: now also U17. (TX)
- net at U5. (SDA/CANL): now also U6. (SDA/CANL); no longer U4. (SDA/CANL)
- net at U5.1 (P1): now also J8.1 (Pin_1); no longer U4.1 (P1)
- net at U6. (SDA/CANL): now also U7. (SDA/CANL); no longer U5. (SDA/CANL)
- net at U6.1 (P1): now also U7.1 (P1); no longer U5.1 (P1)
- net at U9. (SDA/CANL): now also U8. (SDA/CANL)
- net at U8. (SDA/CANL): now also U7. (SDA/CANL); no longer U9. (SDA/CANL)
- net at U9.1 (P1): now also J12.1 (Pin_1)
- net at U8.1 (P1): now also U7.1 (P1); no longer U9.1 (P1)
- new net: U4. (SDA/CANL), U5. (SDA/CANL) (x5)
- new net: U12. (UART_TX), U4. (SDA/CANL) (x2)
- new net: U4.1 (P1), U5.1 (P1) (x2)
- new net: U5. (SDA/CANL), U6. (SDA/CANL) (x4)
- new net: U5.1 (P1), U6.1 (P1) (x2)
- new net: U8. (SDA/CANL), U9. (SDA/CANL) (x4)
- new net: U8.1 (P1), U9.1 (P1) (x2)
- new net: U6. (SDA/CANL), U7. (SDA/CANL) (x4)
- new net: U7. (SDA/CANL), U8. (SDA/CANL) (x4)
- new net: U6.1 (P1), U7.1 (P1)
- new net: U7.1 (P1), U8.1 (P1)
- new net +5V: U17. (TX)
- new net RLCS_ETH: U17. (TX)
- no-connect marks 7 -> 8
Other:
- note added: "PUSR USR-TCP232-T2"
